File: KiCad_flex_PCBs/halbach_45mT_gradient_set/Y_gradient.kicad_pcb (KiCad board)
At the start: 2 copper layers, 217.6 x 125.7 mm, 70 parts, among them J1 SolderPad, J2 SolderPad

Commit message: Add alignment marks and gradient polarity labels to flex PCB export
- axis_marks: axial F.SilkS lines where the rolled coil faces a given
  direction (used for -X left / +X right of the Halbach bore)
- axial_label: +Z bore direction arrows
- positive_gradient: pads labelled so current into the '+' pad gives a
  positive gradient (Y coil is J2+)

Co-Authored-By: Claude Opus 5.5 <noreply@anthropic.com>
Parts:
- removed J1, J2: SolderPad, CoilGen:SolderPad
- added J1-: SolderPad, CoilGen:SolderPad, F.Cu at (13.8, 12.8)
- added J2+: SolderPad, CoilGen:SolderPad, B.Cu at (13.8, 12.8)
Other:
- board text added: "+X RIGHT (looking down +Z)"
- board text added: "+Z into bore -->"
- board text added: "-X LEFT (looking down +Z)"
- board text added: "J1- outside, J2+ inside"
Changed lines of the file:
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@@
 		(layer "F.Cu")
 		(at 13.7500 12.7500)
-		(property "Reference" "J1"
+		(property "Reference" "J1-"
 			(at 0 -2.250 0)
 			(layer "F.Fab")
@@
 		(layer "B.Cu")
 		(at 13.7500 12.7500)
-		(property "Reference" "J2"
+		(property "Reference" "J2+"
 			(at 0 -2.250 0)
 			(layer "B.Fab")
@@
 		)
 	)
+	(gr_line
+		(start 68.7644 134.6946)
+		(end 68.7644 11.0000)
+		(stroke
+			(width 0.3)
+			(type solid)
+		)
+		(layer "F.SilkS")
+	)
+	(gr_line
+		(start 174.7931 134.6946)
+		(end 174.7931 11.0000)
+		(stroke
+			(width 0.3)
+			(type solid)
+		)
+		(layer "F.SilkS")
+	)
+	(gr_text "-X LEFT (looking down +Z)"
+		(at 69.9644 131.6946 90)
+		(layer "F.SilkS")
+		(effects
+			(font
+				(size 1.5 1.5)
+				(thickness 0.225)
+			)
+			(justify left)
+		)
+	)
+	(gr_text "-X LEFT (looking down +Z)"
+		(at 69.9644 68.8473 90)
+		(layer "F.SilkS")
+		(effects
+			(font
+				(size 1.5 1.5)
+				(thickness 0.225)
+			)
+			(justify left)
+		)
+	)
+	(gr_text "+X RIGHT (looking down +Z)"
+		(at 175.9931 131.6946 90)
+		(layer "F.SilkS")
+		(effects
+			(font
+				(size 1.5 1.5)
+				(thickness 0.225)
+			)
+			(justify left)
+		)
+	)
+	(gr_text "+X RIGHT (looking down +Z)"
+		(at 175.9931 68.8473 90)
+		(layer "F.SilkS")
+		(effects
+			(font
+				(size 1.5 1.5)
+				(thickness 0.225)
+			)
+			(justify left)
+		)
+	)
+	(gr_text "+Z into bore -->"
+		(at 19.0000 131.6946 90)
+		(layer "F.SilkS")
+		(effects
+			(font
+				(size 1.5 1.5)
+				(thickness 0.225)
+			)
+			(justify left)
+		)
+	)
+	(gr_text "+Z into bore -->"
+		(at 224.5575 131.6946 90)
+		(layer "F.SilkS")
+		(effects
+			(font
+				(size 1.5 1.5)
+				(thickness 0.225)
+			)
+			(justify left)
+		)
+	)
+	(gr_text "J1- outside, J2+ inside"
+		(at 18.0000 16.5000 0)
+		(layer "F.SilkS")
+		(effects
+			(font
+				(size 1 1)
+				(thickness 0.15)
+			)
+			(justify left)
+		)
+	)
