File: KiCad_flex_PCBs/halbach_45mT_gradient_set/Z_gradient_bore_axis.kicad_pcb (KiCad board)
At the start: 2 copper layers, 209.7 x 123 mm, 70 parts, among them J1 SolderPad, J2 SolderPad

Commit message: Add alignment marks and gradient polarity labels to flex PCB export
- axis_marks: axial F.SilkS lines where the rolled coil faces a given
  direction (used for -X left / +X right of the Halbach bore)
- axial_label: +Z bore direction arrows
- positive_gradient: pads labelled so current into the '+' pad gives a
  positive gradient (Y coil is J2+)

Co-Authored-By: Claude Opus 5.5 <noreply@anthropic.com>
Parts:
- removed J1, J2: SolderPad, CoilGen:SolderPad
- added J1+: SolderPad, CoilGen:SolderPad, F.Cu at (13.8, 72.2)
- added J2-: SolderPad, CoilGen:SolderPad, B.Cu at (13.8, 72.2)
Other:
- board text added: "+X RIGHT (looking down +Z)"
- board text added: "+Z into bore -->"
- board text added: "-X LEFT (looking down +Z)"
- board text added: "J1+ outside, J2- inside"
Changed lines of the file:
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@@
 		(layer "F.Cu")
 		(at 13.7500 72.1903)
-		(property "Reference" "J1"
+		(property "Reference" "J1+"
 			(at 0 -2.250 0)
 			(layer "F.Fab")
@@
 		(layer "B.Cu")
 		(at 13.7500 72.1903)
-		(property "Reference" "J2"
+		(property "Reference" "J2-"
 			(at 0 -2.250 0)
 			(layer "B.Fab")
@@
 		)
 	)
+	(gr_line
+		(start 168.9026 132.0000)
+		(end 168.9026 11.0000)
+		(stroke
+			(width 0.3)
+			(type solid)
+		)
+		(layer "F.SilkS")
+	)
+	(gr_line
+		(start 66.8009 132.0000)
+		(end 66.8009 11.0000)
+		(stroke
+			(width 0.3)
+			(type solid)
+		)
+		(layer "F.SilkS")
+	)
+	(gr_text "-X LEFT (looking down +Z)"
+		(at 170.1026 129.0000 90)
+		(layer "F.SilkS")
+		(effects
+			(font
+				(size 1.5 1.5)
+				(thickness 0.225)
+			)
+			(justify left)
+		)
+	)
+	(gr_text "-X LEFT (looking down +Z)"
+		(at 170.1026 67.5000 90)
+		(layer "F.SilkS")
+		(effects
+			(font
+				(size 1.5 1.5)
+				(thickness 0.225)
+			)
+			(justify left)
+		)
+	)
+	(gr_text "+X RIGHT (looking down +Z)"
+		(at 68.0009 129.0000 90)
+		(layer "F.SilkS")
+		(effects
+			(font
+				(size 1.5 1.5)
+				(thickness 0.225)
+			)
+			(justify left)
+		)
+	)
+	(gr_text "+X RIGHT (looking down +Z)"
+		(at 68.0009 67.5000 90)
+		(layer "F.SilkS")
+		(effects
+			(font
+				(size 1.5 1.5)
+				(thickness 0.225)
+			)
+			(justify left)
+		)
+	)
+	(gr_text "+Z into bore -->"
+		(at 19.0000 129.0000 90)
+		(layer "F.SilkS")
+		(effects
+			(font
+				(size 1.5 1.5)
+				(thickness 0.225)
+			)
+			(justify left)
+		)
+	)
+	(gr_text "+Z into bore -->"
+		(at 216.7035 129.0000 90)
+		(layer "F.SilkS")
+		(effects
+			(font
+				(size 1.5 1.5)
+				(thickness 0.225)
+			)
+			(justify left)
+		)
+	)
+	(gr_text "J1+ outside, J2- inside"
+		(at 18.0000 75.9403 0)
+		(layer "F.SilkS")
+		(effects
+			(font
+				(size 1 1)
+				(thickness 0.15)
+			)
+			(justify left)
+		)
+	)
